File: eagle/led_controller.sch (EAGLE design)
At the start: 12 parts, among them IC1 MC78M05CTG, M1 ARDUINO-NANO-3.0, Q1 TIP120, Q2 TIP120, Q3 TIP120

Commit message: [Eagle] Create new board
Connections:
- net GND: now also M1.GND.1
Changed lines of the file:
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@@
 <class number="0" name="default" width="0" drill="0">
+</class>
+<class number="1" name="3apm" width="2.54" drill="0">
 </class>
 </classes>
@@
 <part name="P+6" library="supply1" deviceset="+12V" device=""/>
 <part name="GND7" library="supply1" deviceset="GND" device=""/>
+<part name="GND8" library="supply1" deviceset="GND" device=""/>
 </parts>
 <sheets>
@@
 <instance part="GND2" gate="1" x="71.12" y="25.4"/>
 <instance part="GND3" gate="1" x="71.12" y="43.18"/>
-<instance part="GND4" gate="1" x="132.08" y="48.26" rot="R90"/>
+<instance part="GND4" gate="1" x="129.54" y="48.26" rot="R90"/>
 <instance part="P+1" gate="1" x="63.5" y="68.58" rot="R270"/>
-<instance part="P+2" gate="1" x="132.08" y="43.18" rot="R270"/>
+<instance part="P+2" gate="1" x="129.54" y="43.18" rot="R270"/>
 <instance part="IQRF" gate="G$1" x="106.68" y="-15.24" rot="R90"/>
 <instance part="P+3" gate="1" x="121.92" y="-7.62" rot="R270"/>
@@
 <instance part="P+6" gate="1" x="53.34" y="-12.7" rot="R180"/>
 <instance part="GND7" gate="1" x="63.5" y="0" rot="R90"/>
+<instance part="GND8" gate="1" x="83.82" y="43.18" rot="R270"/>
 </instances>
 <busses>
@@
 <pinref part="M1" gate="G$1" pin="GND.2"/>
 <pinref part="GND4" gate="1" pin="GND"/>
-<wire x1="129.54" y1="48.26" x2="124.46" y2="48.26" width="0.1524" layer="91"/>
+<wire x1="127" y1="48.26" x2="124.46" y2="48.26" width="0.1524" layer="91"/>
 </segment>
 <segment>
@@
 <pinref part="GND7" gate="1" pin="GND"/>
 </segment>
+<segment>
+<pinref part="M1" gate="G$1" pin="GND.1"/>
+<pinref part="GND8" gate="1" pin="GND"/>
+</segment>
 </net>
 <net name="+5V" class="0">
@@
 <pinref part="M1" gate="G$1" pin="5V"/>
 <pinref part="P+2" gate="1" pin="+5V"/>
-<wire x1="129.54" y1="43.18" x2="124.46" y2="43.18" width="0.1524" layer="91"/>
+<wire x1="127" y1="43.18" x2="124.46" y2="43.18" width="0.1524" layer="91"/>
 </segment>
 <segment>
@@
 </segment>
 </net>
-<net name="+12V" class="0">
+<net name="+12V" class="1">
 <segment>
 <pinref part="P+1" gate="1" pin="+12V"/>
@@
 </segment>
 </net>
-<net name="N$11" class="0">
+<net name="N$11" class="1">
 <segment>
 <pinref part="J1" gate="G$1" pin="3"/>
